File: hw/PiGUS.kicad_sch (KiCad schematic)
At the start: 14 parts, among them J1 IRQDMA_JP, J2 Conn_02x31_Top_Bottom, J3 Bus_ISA_8bit, U1 TXS0108EPW, U2 TXS0108EPW, U3 TXS0108EPW

Commit message: PiGUS Maximus
Parts:
- removed C4: 0.1uF, Capacitor_SMD:C_0805_2012Metric, symbol Device:C
- removed U1, U3: TXS0108EPW, Package_SO:TSSOP-20_4.4x6.5mm_P0.65mm, symbol Logic_LevelTranslator:TXS0108EPW
- added C10, C11: 10uF, Capacitor_THT:CP_Radial_D5.0mm_P2.00mm, symbol Device:C_Polarized_US
- added C7, C8: 0.1uF, Capacitor_SMD:C_0805_2012Metric, symbol Device:C
- added C9: 10u, Capacitor_SMD:C_0805_2012Metric, symbol Device:C
- added D1: LED Green, LED_SMD:LED_0603_1608Metric, symbol Device:LED
- added H1, H2: MountingHole_3.2mm_M3_Pad, MountingHole:MountingHole_3.2mm_M3_Pad, symbol Mechanical:MountingHole_Pad
- added I2S_DAC1: I2S_DAC, PiGUS library:GY-PCM5102, symbol Connector:Conn_01x15_Male
- added J5: ComputeModule4-CM4, CM4IO:Raspberry-Pi-4-Compute-Module, symbol CM4IO:ComputeModule4-CM4
- added J6: Micro_SD_Card, PiGUS library:1140084168, symbol Connector:Micro_SD_Card
- added J7: USB_OTG, Connector_USB:USB_Micro-B_Amphenol_10118194_Horizontal, symbol Connector:USB_OTG
- added J8, J9: eMMC_Boot, Connector_PinHeader_2.54mm:PinHeader_1x02_P2.54mm_Vertical, symbol Connector:Conn_01x02_Male
- added R2: 12K 1%, Resistor_SMD:R_0805_2012Metric, symbol Device:R
- added R3: 1k, Resistor_SMD:R_0603_1608Metric, symbol Device:R
- added U10: TPD2EUSB30, Package_TO_SOT_SMD:Texas_DRT-3, symbol Power_Protection:TPD2EUSB30
- added U3, U4: SN74CB3T3257, Package_SO:TSSOP-16_4.4x5mm_P0.65mm, symbol PiGUS library:74FST3257DR2G
- added U5: 74LVC04, Package_SO:SOIC-14_3.9x8.7mm_P1.27mm, symbol 74xx:74LS04
- added U6: 74LVC00, Package_SO:SOIC-14_3.9x8.7mm_P1.27mm, symbol 74xx:74LS00
- added U7: Pico, PiGUS library:RPi_Pico_SMD_TH, symbol PiGUS library:Pico
- added U8: ESP-PSRAM32, Package_SO:SOIC-8_3.9x4.9mm_P1.27mm, symbol Memory_RAM:ESP-PSRAM32
- added U9: RT9742GGJ5, Package_TO_SOT_SMD:SOT-23-5, symbol CM4IO:RT9742GGJ5
- RPi1: renamed from RPi; footprint Connector_PinSocket_2.54mm:PinSocket_2x20_P2.54mm_Vertical -> Module:Raspberry_Pi_Zero_Socketed_THT_FaceDown_MountingHoles
- renumbered C2 to C1, C1 to C3, C3 to C4, U2 to U1
Connections:
- net RA0 is gone; now on net RA8: RPi1.32 (PWM0/GPIO12)
- net RA1 is gone; now on net RA9: RPi1.33 (PWM1/GPIO13)
- net A0: now also U3.2 (1B1)
- net A1: now also U3.5 (2B1)
- net A2: now also U3.11 (3B1)
- net A3: now also U3.14 (4B1)
- net A4: now also U4.2 (1B1)
- net A5: now also U4.5 (2B1)
- net A6: now also U4.14 (4B1)
- net A7: now also U4.11 (3B1)
- net BUSOE: now also J5.48 (GPIO27), U5.1, U7.34 (GPIO28_ADC2)
- net D0: now also U3.3 (1B2)
- net D1: now also U3.6 (2B2)
- net D2: now also U3.10 (3B2)
- net D3: now also U3.13 (4B2)
- net D4: now also U4.3 (1B2)
- net D5: now also U4.6 (2B2)
- net D6: now also U4.13 (4B2)
- net D7: now also U4.10 (3B2)
- net DACK: now also U6.2
- net GND: now also C10.2, C11.2, C7.2, C8.2, C9.2, H1.1, H2.1, I2S_DAC1.1 (Pin_1), I2S_DAC1.12 (Pin_12), I2S_DAC1.14 (Pin_14), I2S_DAC1.5 (Pin_5), J5.1 (GND), J5.107 (GND), J5.108 (GND), J5.113 (GND), J5.114 (GND), J5.119 (GND), J5.120 (GND), J5.125 (GND), J5.126 (GND), J5.13 (GND), J5.131 (GND), J5.132 (GND), J5.137 (GND), J5.138 (GND), J5.14 (GND), J5.144 (GND), J5.150 (GND), J5.155 (GND), J5.156 (GND), J5.161 (GND), J5.162 (GND), J5.167 (GND), J5.168 (GND), J5.173 (GND), J5.174 (GND), J5.179 (GND), J5.180 (GND), J5.185 (GND), J5.186 (GND), J5.191 (GND), J5.192 (GND), J5.197 (GND), J5.198 (GND), J5.2 (GND), J5.22 (GND), J5.23 (GND), J5.32 (GND), J5.33 (GND), J5.42 (GND), J5.43 (GND), J5.52 (GND), J5.53 (GND), J5.59 (GND), J5.60 (GND), J5.65 (GND), J5.66 (GND), J5.7 (GND), J5.71 (GND), J5.74 (GND), J5.8 (GND), J5.98 (GND), J6.10 (SHIELD), J6.11 (SHIELD), J6.12 (SHIELD), J6.6 (VSS), J6.9 (SHIELD), J7.5 (GND), J7.6 (Shield), J8.1 (Pin_1), U10.3 (GND), U3.8 (GND), U4.8 (GND), U5.7 (GND), U6.7 (GND), U7.13 (GND), U7.18 (GND), U7.23 (GND), U7.28 (GND), U7.3 (GND), U7.33 (AGND), U7.38 (GND), U7.42 (GND), U7.8 (GND), U8.3 (SIO2), U8.4 (VSS), U8.7 (SIO3), U9.2 (GND); no longer J2.42 (Pin_42), J3.42 (AEN)
- net RA8: now also J5.31 (GPIO12), U7.19 (GPIO14); no longer RPi1.38 (GPIO20/MOSI1)
- net RA9: now also J5.28 (GPIO13), U7.20 (GPIO15); no longer RPi1.40 (GPIO21/SCLK1)
- net RDACK: now also J5.47 (GPIO23), U7.26 (GPIO20)
- net RDRQ: now also J5.45 (GPIO24), U7.27 (GPIO21)
- net RIRQ: now also J5.46 (GPIO22), U7.25 (GPIO19)
- net RTC: now also J5.41 (GPIO25), U7.29 (GPIO22)
- net I/OCHRDY: now reaches J2.41 (Pin_41), J3.41 (IO_READY)
- net I/OCHRDY: now also U1.16 (B4)
- net ADS: now reaches RPi1.37 (GPIO26)
- net ADS: now also J5.24 (GPIO26), U3.1 (S), U4.1 (S), U7.32 (GPIO27_ADC1)
- net RA2: no longer names the net of RPi1.8 (GPIO14/TXD)
- net RA3: no longer names the net of RPi1.10 (GPIO15/RXD)
- net RA4: no longer names the net of RPi1.36 (GPIO16)
- net RA5 renamed RI/OCHRDY
- net RI/OCHRDY: now also U1.5 (A4), J5.50 (GPIO17), U7.31 (GPIO26_ADC0)
- net RA6 renamed BCK
- net BCK: now also I2S_DAC1.2 (Pin_2), J5.49 (GPIO18), U7.21 (GPIO16)
- net RA7 renamed DIN
- net DIN: now also I2S_DAC1.3 (Pin_3), J5.26 (GPIO19), U7.22 (GPIO17)
- net RD0 renamed AD0
- net AD0: now also J5.54 (GPIO4), U3.4 (1A), U7.9 (GPIO6)
- net RD1 renamed AD1
- net AD1: now also J5.34 (GPIO5), U3.7 (2A), U7.10 (GPIO7)
- net RD2 renamed AD2
- net AD2: now also J5.30 (GPIO6), U3.9 (3A), U7.11 (GPIO8)
- net RD3 renamed AD3
- net AD3: now also J5.37 (GPIO7), U3.12 (4A), U7.12 (GPIO9)
- net RD4 renamed AD4
- net AD4: now also J5.39 (GPIO8), U4.4 (1A), U7.14 (GPIO10)
- net RD5 renamed AD5
- net AD5: now also J5.40 (GPIO9), U4.7 (2A), U7.15 (GPIO11)
- net RD6 renamed AD6
- net AD6: now also J5.44 (GPIO10), U4.9 (3A), U7.16 (GPIO12)
- net RD7 renamed AD7
- net AD7: now also J5.38 (GPIO11), U4.12 (4A), U7.17 (GPIO13)
- net RnIOR renamed ~{RIOR}
- net ~{RIOR}: now also J5.35 (ID_SC), U6.8, U7.2 (GPIO1); no longer U1.5 (A4)
- net RnIOW: no longer names the net of U1.4 (A3)
- net RnIOW: no longer RPi1.27 (ID_SD/GPIO0)
- net VCC renamed +5V
- net +5V: now also C10.1, I2S_DAC1.6 (Pin_6), J5.77 (+5v_(Input)), J5.79 (+5v_(Input)), J5.81 (+5v_(Input)), J5.83 (+5v_(Input)), J5.85 (+5v_(Input)), J5.87 (+5v_(Input)), J9.1 (Pin_1), U7.39 (VSYS); no longer C6.1
- net VCC33 renamed +3V3
- net +3V3: now also C6.1, C11.1, C7.1, C8.1, D1.2 (A), J5.78 (GPIO_VREF(1.8v/3.3v_Input)), J5.84 (+3.3v_(Output)), J5.86 (+3.3v_(Output)), R2.1, U3.16 (VCC), U4.16 (VCC), U5.11, U5.13, U5.14 (VCC), U5.9, U6.12, U6.13, U6.14 (VCC), U7.36 (3V3), U8.8 (VCC), U9.5 (IN)
- net nIOR renamed ~{IOR}
- net ~{IOR}: now also U5.3; no longer U1.16 (B4)
- net nIOW renamed ~{IOW}
- net ~{IOW}: now also U5.5; no longer U1.17 (B3)
- new net: D1.1 (K), R3.1
- new net: J7.1 (VBUS), J9.2 (Pin_2)
- new net: U5.6, U6.5
- new net: U5.4, U6.9
- new net: U6.10, U6.3, U6.4
- new net: J5.93 (nRPIBOOT), J8.2 (Pin_2)
- new net AEN: J2.42 (Pin_42), J3.42 (AEN), U6.1
- new net CM4_Activity: J5.21 (PI_nLED_Activity), R3.2
- new net LRCK: I2S_DAC1.4 (Pin_4), J5.25 (GPIO21), RPi1.40 (GPIO21/SCLK1), U7.24 (GPIO18)
- new net SD_CLK: J5.57 (SD_CLK), J6.5 (CLK)
- new net SD_CMD: J5.62 (SD_CMD), J6.3 (CMD)
- new net SD_DAT0: J5.63 (SD_DAT0), J6.7 (DAT0)
- new net SD_DAT1: J5.67 (SD_DAT1), J6.8 (DAT1)
- new net SD_DAT2: J5.69 (SD_DAT2), J6.1 (DAT2)
- new net SD_DAT3: J5.61 (SD_DAT3), J6.2 (DAT3/CD)
- new net SD_PWR: C9.1, J6.4 (VDD), U9.1 (OUT)
- new net SD_PWR_ON: R2.2, U9.4 (EN)
- new net SPI_RX: U7.6 (GPIO4), U8.2 (SO/SIO)
- new net SPI_SCK: U7.4 (GPIO2), U8.6 (SCLK)
- new net SPI_TX: U7.5 (GPIO3), U8.5 (SI/SIO)
- new net USB2_N: J5.103 (USB2_N), J7.2 (D-), U10.2 (D-)
- new net USB2_P: J5.105 (USB2_P), J7.3 (D+), U10.1 (D+)
- new net ~{BUSOE}: U3.15 (~{OE}), U4.15 (~{OE}), U5.2
- new net ~{RIOW}: J5.36 (ID_SD), RPi1.27 (ID_SD/GPIO0), U6.6, U7.1 (GPIO0)
- new net ~{SPI_CS}: U7.7 (GPIO5), U8.1 (~{CE})
- no-connect marks 0 -> 137
Other:
- note added: "Activity LED"
- moved on the sheet: C1, C3, C4, C5, J1, J2, J3, R1, RPi1, U1
